Commit message: wygenerowanie mapy

File: src/vizualization_map/mapa.urdf (robot description, URDF)
Before this commit: robot lights, 34 links, 33 joints
Links:
- link road_1_2: geometry visual box size=250 4 0.1
- link road_1_4: geometry visual box size=4 200 0.1
- link road_2_3: geometry visual box size=300 4 0.1
- link road_2_5: geometry visual box size=4 200 0.1
- link road_3_7: geometry visual box size=4 200 0.1
- link road_4_5: geometry visual box size=250 4 0.1
- link road_4_8: geometry visual box size=4 150 0.1
- link road_5_6: geometry visual box size=100 4 0.1
- link road_5_9: geometry visual box size=4 150 0.1
- link road_6_10: geometry visual box size=4 150 0.1
- link road_6_7: geometry visual box size=200 4 0.1
- link road_8_9: geometry visual box size=250 4 0.1
- link road_9_10: geometry visual box size=100 4 0.1
Joints:
- joint cross_base_to_link_10: origin xyz=360 360 0.01 rpy=0 0 0 -> xyz=350 -350 0.01 rpy=0 0 0
- joint cross_base_to_link_2: origin xyz=0 255 0.01 rpy=0 0 0 -> xyz=250 0 0.01 rpy=0 0 0
- joint cross_base_to_link_3: origin xyz=0 560 0.01 rpy=0 0 0 -> xyz=550 0 0.01 rpy=0 0 0
- joint cross_base_to_link_4: origin xyz=205 0 0.01 rpy=0 0 0 -> xyz=0 -200 0.01 rpy=0 0 0
- joint cross_base_to_link_5: origin xyz=205 255 0.01 rpy=0 0 0 -> xyz=250 -200 0.01 rpy=0 0 0
- joint cross_base_to_link_6: origin xyz=205 360 0.01 rpy=0 0 0 -> xyz=350 -200 0.01 rpy=0 0 0
- joint cross_base_to_link_7: origin xyz=205 560 0.01 rpy=0 0 0 -> xyz=550 -200 0.01 rpy=0 0 0
- joint cross_base_to_link_8: origin xyz=360 0 0.01 rpy=0 0 0 -> xyz=0 -350 0.01 rpy=0 0 0
- joint cross_base_to_link_9: origin xyz=360 255 0.01 rpy=0 0 0 -> xyz=250 -350 0.01 rpy=0 0 0
- joint road_1_2_to_cross: origin xyz=0 127 0 rpy=0 0 0 -> xyz=125 0 0 rpy=0 0 0
- joint road_1_4_to_cross: origin xyz=102 0 0 rpy=0 0 0 -> xyz=0 -100 0 rpy=0 0 0
- joint road_2_3_to_cross: origin xyz=0 152 0 rpy=0 0 0 -> xyz=150 0 0 rpy=0 0 0
- joint road_2_5_to_cross: origin xyz=102 0 0 rpy=0 0 0 -> xyz=0 -100 0 rpy=0 0 0
- joint road_3_7_to_cross: origin xyz=102 0 0 rpy=0 0 0 -> xyz=0 -100 0 rpy=0 0 0
- joint road_4_5_to_cross: origin xyz=0 127 0 rpy=0 0 0 -> xyz=125 0 0 rpy=0 0 0
- joint road_4_8_to_cross: origin xyz=77 0 0 rpy=0 0 0 -> xyz=0 -75 0 rpy=0 0 0
- joint road_5_6_to_cross: origin xyz=0 52 0 rpy=0 0 0 -> xyz=50 0 0 rpy=0 0 0
- joint road_5_9_to_cross: origin xyz=77 0 0 rpy=0 0 0 -> xyz=0 -75 0 rpy=0 0 0
- joint road_6_10_to_cross: origin xyz=77 0 0 rpy=0 0 0 -> xyz=0 -75 0 rpy=0 0 0
- joint road_6_7_to_cross: origin xyz=0 100 0 rpy=0 0 0 -> xyz=100 0 0 rpy=0 0 0
- joint road_8_9_to_cross: origin xyz=0 127 0 rpy=0 0 0 -> xyz=125 0 0 rpy=0 0 0
- joint road_9_10_to_cross: origin xyz=0 52 0 rpy=0 0 0 -> xyz=50 0 0 rpy=0 0 0
